File: IFTENDO.kicad_pcb (KiCad board)
At the start: 2 copper layers, 54 x 85.6 mm, 11 parts, among them J1 Conn_01x10_Pin, J2 Conn_01x10_Pin, J3 Conn_01x04_Socket

Commit message: Version sent to aisler for production
Parts:
- added D1: 1N4148WS, Diode_SMD:D_SOD-323_HandSoldering, F.Cu at (110.1, 68.9)
- added D2: 1N4148WS, Diode_SMD:D_SOD-323_HandSoldering, F.Cu at (110.1, 71.5)
- added D3: 1N4148WS, Diode_SMD:D_SOD-323_HandSoldering, F.Cu at (110.1, 74.0)
- added D4: 1N4148WS, Diode_SMD:D_SOD-323_HandSoldering, F.Cu at (110.1, 76.6)
- added D5: 1N4148WS, Diode_SMD:D_SOD-323_HandSoldering, F.Cu at (110.1, 84.2)
- added D6: 1N4148WS, Diode_SMD:D_SOD-323_HandSoldering, F.Cu at (110.1, 79.1)
- added D7: 1N4148WS, Diode_SMD:D_SOD-323_HandSoldering, F.Cu at (110.0, 81.6)
- added D8: 1N4148WS, Diode_SMD:D_SOD-323_HandSoldering, F.Cu at (110.1, 86.7)
- added D9: LED, Diode_SMD:D_0805_2012Metric_Pad1.15x1.40mm_HandSolder, F.Cu at (81.7, 51.0)
- added G***: LOGO, Local footprints:Logo_texte_DVIC_kicad_mask_12mm, F.Cu at (83.7, 122.6)
- added G***: LOGO, Local footprints:logo_IFT_12mm, F.Cu at (121.2, 50.1)
- added G***: LOGO, Local footprints:Logo_IFT_50mm_silk, B.Cu at (100.6, 106.8)
- added R1: 10K, Resistor_SMD:R_0805_2012Metric_Pad1.20x1.40mm_HandSolder, F.Cu at (81.7, 54.0)
- moved S5 7.83 mm to (114.2, 103.4), turned to 90 degrees
- moved S6 3.07 mm to (124.1, 99.2), turned to 90 degrees
- moved S4 2.95 mm to (88.2, 111.3)
- moved S1 2.81 mm to (80.2, 103.3)
- moved S3 2.36 mm to (88.2, 95.3)
- moved S2 2.28 mm to (96.2, 103.3)
- moved S8 1.92 mm to (110.2, 123.2), turned to 180 degrees
- moved S7 1.34 mm to (97.4, 123.2), turned to 180 degrees
Connections:
- net /Button5/NO renamed /ButtonB/NO
- net /Button7/NO renamed /ButtonSelect/NO
- net /Button8/NO renamed /ButtonStart/NO
- net /button_A renamed /ButtonA/NO
- net /button_U renamed /ButtonUp/NO
- J1 pad 1: /GPIO0 -> /RGB_OUT
- J1 pad 10: +3.3V -> unconnected-(J1-Pin_10-Pad10)
- J1 pad 2: /GPIO1 -> /GPIO4
- J1 pad 3: /GPIO2 -> /GPIO5
- J1 pad 4: /GPIO3 -> /GPIO6
- J1 pad 5: /GPIO10 -> /GPIO7
- J1 pad 6: /Tx -> /GPIO8
- J1 pad 7: /Rx -> /GPIO9
- J2 pad 1: unconnected-(J2-Pin_1-Pad1) -> +3.3V
- J2 pad 10: /RGB_OUT -> /GPIO0
- J2 pad 4: /GPIO9 -> /O_1
- J2 pad 5: /GPIO8 -> /Tx
- J2 pad 6: /GPIO7 -> /GPIO10
- J2 pad 7: /GPIO6 -> /GPIO3
- J2 pad 8: /GPIO5 -> /GPIO2
- J2 pad 9: /GPIO4 -> /GPIO1
- J3 pad 3: /SCK -> /GPIO6
- J3 pad 4: /SDA -> /GPIO5
- S1 pad 1: GND -> /O_1
- S1 pad 2: GND -> /O_1
- S1 pad 3: /GPIO4 -> /ButtonLeft/NO
- S1 pad 4: /GPIO4 -> /ButtonLeft/NO
- S2 pad 1: GND -> /GPIO10
- S2 pad 2: GND -> /GPIO10
- S2 pad 3: /GPIO6 -> /ButtonRight/NO
- S2 pad 4: /GPIO6 -> /ButtonRight/NO
- S3 pad 1: GND -> /O_1
- S3 pad 2: GND -> /O_1
- S4 pad 1: GND -> /O_1
- S4 pad 2: GND -> /O_1
- S4 pad 3: /GPIO5 -> /ButtonDown/NO
- S4 pad 4: /GPIO5 -> /ButtonDown/NO
- S5 pad 1: GND -> /GPIO0
- S5 pad 2: GND -> /GPIO0
- S6 pad 1: GND -> /GPIO0
- S6 pad 2: GND -> /GPIO0
- S7 pad 1: GND -> /GPIO10
- S7 pad 2: GND -> /GPIO10
- S8 pad 1: GND -> /GPIO10
- S8 pad 2: GND -> /GPIO10
Routing:
- net /GPIO10: track 0.00 -> 85.5 mm, vias 0 -> 2
- net /GPIO0: track 0.00 -> 81.6 mm, vias 0 -> 1
- net /O_1: track 0.00 -> 58.8 mm
- net /ButtonLeft/NO: track 0.00 -> 55.0 mm
- net /ButtonDown/NO: track 0.00 -> 49.2 mm
- net /ButtonRight/NO: track 0.00 -> 47.2 mm
- net /ButtonSelect/NO: track 0.00 -> 46.7 mm
- net /ButtonB/NO: track 0.00 -> 42.2 mm
- net /ButtonStart/NO: track 0.00 -> 41.8 mm
- net /ButtonA/NO: track 0.00 -> 41.6 mm
- net /ButtonUp/NO: track 0.00 -> 41.5 mm
- net +3.3V: track 0.00 -> 38.1 mm
- net /Tx: track 0.00 -> 24.7 mm
- net /GPIO8: track 0.00 -> 22.8 mm
- net /GPIO6: track 0.00 -> 21.4 mm
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Other:
- board text added: "+3V3"
- board text added: "A"
- board text added: "B"
- board text added: "Down"
- board text added: "GND"
- board text added: "IFTENTO Game Board 11/2023"
- board text added: "Left"
- board text added: "Right"
- board text added: "SCL"
- board text added: "SDA"
- board text added: "Select"
- board text added: "Start"
- board text added: "Up"
- board text added: "Vin"
