File: IFTENDO.kicad_sch (KiCad schematic)
At the start: 3 parts, among them J2 Conn_01x10_Pin, J3 Conn_01x04_Socket, J4 Conn_01x10_Pin

Commit message: Version sent to aisler for production
Parts:
- added D1, D2, D3, D4, D5, D6, D7, D8: 1N4148WS, Diode_SMD:D_SOD-323_HandSoldering, symbol Diode:1N4148WS
- added D1: LED, Diode_SMD:D_0805_2012Metric_Pad1.15x1.40mm_HandSolder, symbol Device:LED
- added R1: 10K, Resistor_SMD:R_0805_2012Metric_Pad1.20x1.40mm_HandSolder, symbol Device:R_Small
Connections:
- net Rx is gone; now on net GPIO9: J2.7 (Pin_7)
- net SCK is gone; now on net GPIO6: J3.3 (Pin_3)
- net SDA is gone; now on net GPIO5: J3.4 (Pin_4)
- net +3.3V: now also J4.1 (Pin_1); no longer J2.10 (Pin_10)
- net ButtonB/NO: now also D4.2 (A)
- net ButtonSelect/NO: now also D5.2 (A)
- net ButtonStart/NO: now also D8.2 (A)
- net GND: now also D1.1 (K)
- net GPIO0: now also J4.10 (Pin_10); no longer J2.1 (Pin_1)
- net GPIO1: now also J4.9 (Pin_9); no longer J2.2 (Pin_2)
- net GPIO10: now also J4.6 (Pin_6); no longer J2.5 (Pin_5)
- net GPIO2: now also J4.8 (Pin_8); no longer J2.3 (Pin_3)
- net GPIO3: now also J4.7 (Pin_7); no longer J2.4 (Pin_4)
- net GPIO4: now also J2.2 (Pin_2); no longer J4.9 (Pin_9)
- net GPIO5: now also J2.3 (Pin_3); no longer J4.8 (Pin_8)
- net GPIO6: now also J2.4 (Pin_4); no longer J4.7 (Pin_7)
- net GPIO7: now also J2.5 (Pin_5), D1.1 (K), D2.1 (K), D3.1 (K); no longer J4.6 (Pin_6)
- net GPIO8: now also J2.6 (Pin_6), D4.1 (K), D5.1 (K), D6.1 (K); no longer J4.5 (Pin_5)
- net GPIO9: now also D7.1 (K), D8.1 (K); no longer J4.4 (Pin_4)
- net RGB_OUT: now also J2.1 (Pin_1); no longer J4.10 (Pin_10)
- net Tx: now also J4.5 (Pin_5), R1.1; no longer J2.6 (Pin_6)
- new net: D1.2 (A), R1.2
- new net ButtonA/NO: D3.2 (A)
- new net ButtonDown/NO: D7.2 (A)
- new net ButtonLeft/NO: D6.2 (A)
- new net ButtonRight/NO: D2.2 (A)
- new net ButtonUp/NO: D1.2 (A)
- new net O_1: J4.4 (Pin_4)
- no-connect marks 2 -> 1
Other:
- sheet Button1 renamed ButtonLeft
- sheet Button2 renamed ButtonRight
- sheet Button3 renamed ButtonUp
- sheet Button4 renamed ButtonDown
- sheet Button5 renamed ButtonB
- sheet Button6 renamed ButtonA
- sheet Button7 renamed ButtonSelect
- sheet Button8 renamed ButtonStart
- note added: "Connector to screen"
- note added: "Connectors to µC board (flipped as board will connect from the back side)"
- note added: "Keyboard matrix"
- note removed: "Connectors to µC board"
- company: (none) -> IFT
- title: (none) -> IFTENTO
- moved on the sheet: J2, J4
